Commit message: corona em commit

File: lasmultidescription4/urdf/base_multiple.xacro (robot description, xacro)
@@ -14,5 +14,5 @@
  	       <origin xyz="0 0 0" rpy="0 0 0" />
        	 <geometry>
-             <mesh filename="package://nexus/meshes/base-binary.stl"/>
+             <mesh filename="package://nexus/meshes/base2-binary.stl"/>
        	 </geometry>
  	       <material name="Yellow"/>
@@ -32,4 +32,35 @@
        </inertial>
    </link>
+   <xacro:macro name="cylinder_inertia" params="m r h">
+    <inertial>
+      <mass value="${m}"/>
+      <inertia ixx="${m*(3*r*r+h*h)/12}" ixy = "0" ixz = "0" iyy="${m*(3*r*r+h*h)/12}" iyz = "0" izz="${m*r*r/2}"/>
+    </inertial>
+  </xacro:macro>
+  <xacro:macro name="wheel" params="prefix reflect">
+    <link name="${prefix}_wheel">
+      <visual>
+        <origin xyz="0 0 0" rpy="${pi/2} 0 0"/>
+        <geometry>
+          <cylinder radius="${wheel_radius}" length="0.005"/>
+        </geometry>
+      </visual>
+      <collision>
+        <origin xyz="0 0 0" rpy="${pi/2} 0 0"/>
+        <geometry>
+          <cylinder radius="${wheel_radius}" length="0.005"/>
+        </geometry>
+      </collision>
+      <xacro:cylinder_inertia m="10" r="${wheel_radius}" h="0.005"/>
+    </link>
+    <joint name="${prefix}_wheel_joint" type="continuous">
+      <axis xyz="0 1 0" rpy="0 0 0" />
+      <parent link="base_link"/>
+      <child link="${prefix}_wheel"/>
+      <origin xyz="${wheel_joint_offset} ${((base_width/2)+base_wheel_gap)*reflect} -0.005" rpy="0 0 0"/>
+    </joint>
+  </xacro:macro>
+  <xacro:wheel prefix="left" reflect="1"/>
+  <xacro:wheel prefix="right" reflect="-1"/>
     <gazebo>
       <!-- planar plugin is very simple, it wil ALWAYS force a speed, so if lifted, the object doesn't fall.

File: lasmultidescription4/urdf/robot_base_multiple.xacro (robot description, xacro)
@@ -32,5 +32,5 @@
   </hokuyo_utm30lx_model>
   <imu_model parent="$(arg prefix)base_footprint" name="$(arg prefix)imu" topic="/$(arg prefix)/imu_data" hz="10">
-    <origin xyz="0 0 0.5" rpy="0 0 0" />
+    <origin xyz="0 0 0.42" rpy="0 0 0" />
   </imu_model>
 </robot>

Commit message: improved decentralised ctrler

File: lasmultidescription4/urdf/base_multiple.xacro (robot description, xacro)
@@ -3,4 +3,5 @@
   <xacro:property name="M_PI" value="3.14159"/>
   <xacro:property name="MESH_SCALE" value="100"/>
+  <xacro:property name="wheel_radius" value="0.2"/>
   <xacro:macro name="nexus_body"  params="parent rn *oorsprong">
    <joint name="${rn}base_footprint_joint" type="fixed">
@@ -32,35 +33,4 @@
        </inertial>
    </link>
-   <xacro:macro name="cylinder_inertia" params="m r h">
-    <inertial>
-      <mass value="${m}"/>
-      <inertia ixx="${m*(3*r*r+h*h)/12}" ixy = "0" ixz = "0" iyy="${m*(3*r*r+h*h)/12}" iyz = "0" izz="${m*r*r/2}"/>
-    </inertial>
-  </xacro:macro>
-  <xacro:macro name="wheel" params="prefix reflect">
-    <link name="${prefix}_wheel">
-      <visual>
-        <origin xyz="0 0 0" rpy="${pi/2} 0 0"/>
-        <geometry>
-          <cylinder radius="${wheel_radius}" length="0.005"/>
-        </geometry>
-      </visual>
-      <collision>
-        <origin xyz="0 0 0" rpy="${pi/2} 0 0"/>
-        <geometry>
-          <cylinder radius="${wheel_radius}" length="0.005"/>
-        </geometry>
-      </collision>
-      <xacro:cylinder_inertia m="10" r="${wheel_radius}" h="0.005"/>
-    </link>
-    <joint name="${prefix}_wheel_joint" type="continuous">
-      <axis xyz="0 1 0" rpy="0 0 0" />
-      <parent link="base_link"/>
-      <child link="${prefix}_wheel"/>
-      <origin xyz="${wheel_joint_offset} ${((base_width/2)+base_wheel_gap)*reflect} -0.005" rpy="0 0 0"/>
-    </joint>
-  </xacro:macro>
-  <xacro:wheel prefix="left" reflect="1"/>
-  <xacro:wheel prefix="right" reflect="-1"/>
     <gazebo>
       <!-- planar plugin is very simple, it wil ALWAYS force a speed, so if lifted, the object doesn't fall.
