Commit message: last_day

File: lasmultidescription4/urdf/hokuyo_utm30lx.urdf.xacro (robot description, xacro)
@@ -17,5 +17,5 @@
           <origin xyz="0 0 0" rpy="0 0 0" />
           <geometry>
-            <cylinder length="0.05" radius="0.1"/>
+            <cylinder length="0.05" radius="0.06"/>
           </geometry>
         </visual>
